Commit message: added sim

File: robot_ws/install/ros_gz_h1_description/share/ros_gz_h1_description/models/h1_ign/h1_2.urdf (robot description, URDF)
Before this commit: robot h1_2, 58 links, 57 joints
Links:
- added link head_link, mass 1.0; visual sphere radius=0.08
- added link neck_link, mass 0.5; visual cylinder length=0.05 radius=0.03
Joints:
- added joint neck_pan_joint: type revolute, parent torso_link, child neck_link, origin xyz=0 0 0.65 rpy=0 0 0, axis 0 0 1, limit lower=-1.57 upper=1.57 effort=10.0 velocity=5.0
- added joint neck_tilt_joint: type revolute, parent neck_link, child head_link, origin xyz=0 0 0.025 rpy=0 0 0, axis 0 1 0, limit lower=-0.78 upper=0.78 effort=10.0 velocity=5.0

File: robot_ws/install/ros_gz_h1_description/share/ros_gz_h1_description/models/h1_ign/h1_2_handless.urdf (robot description, URDF)
Before this commit: robot h1_2, 32 links, 31 joints
Links:
- added link head_link, mass 1.0; visual sphere radius=0.08
- added link neck_link, mass 0.5; visual cylinder length=0.05 radius=0.03
Joints:
- added joint neck_pan_joint: type revolute, parent torso_link, child neck_link, origin xyz=0 0 0.65 rpy=0 0 0, axis 0 0 1, limit lower=-1.57 upper=1.57 effort=10.0 velocity=5.0
- added joint neck_tilt_joint: type revolute, parent neck_link, child head_link, origin xyz=0 0 0.025 rpy=0 0 0, axis 0 1 0, limit lower=-0.78 upper=0.78 effort=10.0 velocity=5.0
