Commit message: video

File: robot_ws/install/ros_gz_h1_description/share/ros_gz_h1_description/models/h1_ign/h1_2_handless.urdf (robot description, URDF)
Before this commit: robot h1_2, 34 links, 33 joints
Links:
- link head_link: geometry visual sphere radius=0.1
- link neck_link: geometry visual cylinder length=0.105 radius=0.05
Joints:
- joint neck_pan_joint: origin xyz=0 0 0.65 rpy=0 0 0 -> xyz=0 0 0.55 rpy=0 0 0

Commit message: fixed gazebo crash

File: robot_ws/install/ros_gz_h1_description/share/ros_gz_h1_description/models/h1_ign/h1_2_handless.urdf (robot description, URDF)
Before this commit: robot h1_2, 34 links, 33 joints
Links:
- added link base_link
Joints:
- added joint base_joint: type fixed, parent base_link, child pelvis, origin xyz=0 0 0 rpy=0 0 0
